File: rack/thatmicpre_v2.kicad_pcb (KiCad board)
At the start: 2 copper layers, 140 x 73.6 mm, 88 parts, among them J1 CON-SOCJ-2155, J10 Angled pinheader, J11 NCJ6FA-H, J2 NC3FBH2, J4 Female header, J5 Male pinheader, J6 Female header, J7 Male pinheader, J8 Angled pinheader, Q1 BC546CTA, Q2 BC546CTA, SW1 DPDT, SW2 DPDT, SW3 SR2612F-0112-38F5B-D8-S, U1 1512P08-U

Commit message: Fixed the issue where the 1/2W resistor was not placed correctly; added square pads for connecting to the enclosure.
Parts:
- moved R4 2.29 mm to (144.9, 122.4)
- moved R3 2.29 mm to (148.9, 122.4)
Routing:
- net Net-(D2-K): track 51.3 -> 49.1 mm
- net Net-(C4-Pad2): track 29.5 -> 31.7 mm
- net Net-(C5-Pad2): track 8.17 -> 10.1 mm
- net Net-(SW1B-B): track 122.3 -> 124.0 mm
- net /V35P: track 70.2 -> 68.5 mm
- net Net-(D1-K): track 45.6 -> 44.7 mm
- net /V18P: track 77.6 -> 77.0 mm
